File: KiCAD Part One -2023-02-25_184051/KiCAD Part One .kicad_sch (KiCad schematic)
At the start: 6 parts, among them SW1 

Commit message: EE 201 GerberFile
Parts:
- 2.2kOhm1: renamed from 2.2kOhm; footprint (none) -> Resistor_THT:R_Axial_DIN0516_L15.5mm_D5.0mm_P20.32mm_Horizontal
- C1: footprint (none) -> Capacitor_THT:C_Radial_D5.0mm_H5.0mm_P2.00mm
- D1: footprint (none) -> LED_THT:LED_D5.0mm
- R1: footprint (none) -> Resistor_THT:R_Axial_DIN0516_L15.5mm_D5.0mm_P20.32mm_Horizontal
- SW1: footprint (none) -> Button_Switch_THT:SW_E-Switch_EG1224_SPDT_Angled
- V1: footprint (none) -> Connector_JST:JST_PH_B2B-PH-K_1x02_P2.00mm_Vertical
Changed lines of the file:
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@@
       (effects (font (size 1.27 1.27)) (justify left))
     )
-    (property "Footprint" "" (id 2) (at 174.9552 100.33 0)
+    (property "Footprint" "Capacitor_THT:C_Radial_D5.0mm_H5.0mm_P2.00mm" (id 2) (at 174.9552 100.33 0)
       (effects (font (size 1.27 1.27)) hide)
     )
@@
       (effects (font (size 1.27 1.27)) (justify left))
     )
-    (property "Footprint" "" (id 2) (at 195.072 87.63 90)
+    (property "Footprint" "Resistor_THT:R_Axial_DIN0516_L15.5mm_D5.0mm_P20.32mm_Horizontal" (id 2) (at 195.072 87.63 90)
       (effects (font (size 1.27 1.27)) hide)
     )
@@
   (symbol (lib_id "Device:R") (at 147.32 83.82 270) (unit 1)
     (in_bom yes) (on_board yes)
-    (property "Reference" "2.2kOhm" (id 0) (at 147.32 88.9 90))
+    (property "Reference" "2.2kOhm1" (id 0) (at 147.32 88.9 90))
     (property "Value" "R2" (id 1) (at 147.32 86.36 90))
-    (property "Footprint" "" (id 2) (at 147.32 82.042 90)
+    (property "Footprint" "Resistor_THT:R_Axial_DIN0516_L15.5mm_D5.0mm_P20.32mm_Horizontal" (id 2) (at 147.32 82.042 90)
       (effects (font (size 1.27 1.27)) hide)
     )
@@
     (property "Reference" "V1" (id 0) (at 139.7 90.17 0))
     (property "Value" "9V" (id 1) (at 139.7 92.71 0))
-    (property "Footprint" "" (id 2) (at 132.08 90.17 0)
+    (property "Footprint" "Connector_JST:JST_PH_B2B-PH-K_1x02_P2.00mm_Vertical" (id 2) (at 132.08 90.17 0)
       (effects (font (size 1.27 1.27)) hide)
     )
@@
       (effects (font (size 1.27 1.27)) (justify right))
     )
-    (property "Footprint" "" (id 2) (at 196.85 109.22 0)
+    (property "Footprint" "LED_THT:LED_D5.0mm" (id 2) (at 196.85 109.22 0)
       (effects (font (size 1.27 1.27)) hide)
     )
@@
     (property "Reference" "SW1" (id 0) (at 160.02 86.36 0))
     (property "Value" "  " (id 1) (at 161.29 76.2 0))
-    (property "Footprint" "" (id 2) (at 161.29 81.28 0)
+    (property "Footprint" "Button_Switch_THT:SW_E-Switch_EG1224_SPDT_Angled" (id 2) (at 161.29 81.28 0)
       (effects (font (size 1.27 1.27)) hide)
     )
@@
   (symbol_instances
     (path "/8ee06da2-e8fe-46a6-8c79-9b905d2ea634"
-      (reference "2.2kOhm") (unit 1) (value "R2") (footprint "")
+      (reference "2.2kOhm1") (unit 1) (value "R2") (footprint "Resistor_THT:R_Axial_DIN0516_L15.5mm_D5.0mm_P20.32mm_Horizontal")
     )
     (path "/02ac4cfc-df1f-4916-b880-6eddb351e225"
-      (reference "C1") (unit 1) (value "2.7 uF") (footprint "")
+      (reference "C1") (unit 1) (value "2.7 uF") (footprint "Capacitor_THT:C_Radial_D5.0mm_H5.0mm_P2.00mm")
     )
     (path "/e2cee6fd-a24a-4a32-a65d-9eab07c61240"
-      (reference "D1") (unit 1) (value "    ") (footprint "")
+      (reference "D1") (unit 1) (value "    ") (footprint "LED_THT:LED_D5.0mm")
     )
     (path "/19bc6b6d-a8d1-4fee-9dda-0e0f793cfe6d"
-      (reference "R1") (unit 1) (value "20kOhm") (footprint "")
+      (reference "R1") (unit 1) (value "20kOhm") (footprint "Resistor_THT:R_Axial_DIN0516_L15.5mm_D5.0mm_P20.32mm_Horizontal")
     )
     (path "/f71388fa-db07-4371-836f-6f00000d17f3"
-      (reference "SW1") (unit 1) (value "  ") (footprint "")
+      (reference "SW1") (unit 1) (value "  ") (footprint "Button_Switch_THT:SW_E-Switch_EG1224_SPDT_Angled")
     )
     (path "/a6df68a3-2bea-4546-8176-ddb97d4bd3e8"
-      (reference "V1") (unit 1) (value "9V") (footprint "")
+      (reference "V1") (unit 1) (value "9V") (footprint "Connector_JST:JST_PH_B2B-PH-K_1x02_P2.00mm_Vertical")
     )
   )
