File: KiCAD Part One -2023-02-25_184051/KiCAD Part One .kicad_pcb (KiCad board)
At the start: 2 copper layers, 6 parts, among them SW1 

Commit message: arduino part two
Routing:
- net Net-(C1-Pad1): track 74.5 -> 73.9 mm
- net Net-(C1-Pad2): track 82.8 -> 82.3 mm
Other:
- board outline added: 101.6 x 45.7 mm
Changed lines of the file:
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@@
       (outputformat 1)
       (mirror false)
-      (drillshape 1)
+      (drillshape 0)
       (scaleselection 1)
-      (outputdirectory "")
+      (outputdirectory "/Users/keerthi-personal/Documents/EE201/KiCAD Part One -2023-02-25_184051/")
     )
   )
@@
     (fp_line (start -1.95 2.8) (end 3.95 2.8) (layer "F.Fab") (width 0.1))
     (fp_line (start -1.11 -2.11) (end -2.36 -2.11) (layer "F.Fab") (width 0.1))
-    (pad "1" thru_hole roundrect (at 0 0 270) (size 1.2 1.75) (drill 0.75) (layers *.Cu *.Mask) (roundrect_rratio 0.208333)
+    (pad "1" thru_hole roundrect (at 0 0 270) (size 1.2 1.75) (drill 0.75) (layers *.Cu *.Mask) (roundrect_rratio 0.2083333333)
       (net 2 "Net-(2.2kOhm1-Pad2)") (pinfunction "Pin_1") (pintype "passive"))
     (pad "2" thru_hole oval (at 2 0 270) (size 1.2 1.75) (drill 0.75) (layers *.Cu *.Mask)
@@
     )
   )
+  (gr_rect (start 81.28 78.74) (end 182.88 124.46) (layer "Edge.Cuts") (width 0.1) (fill none))
   (segment (start 111.76 86.36) (end 112.96 87.56) (width 0.25) (layer "F.Cu") (net 1))
   (segment (start 112.96 87.56) (end 127.4325 87.56) (width 0.25) (layer "F.Cu") (net 1))
@@
   (segment (start 91.39 114.3) (end 91.44 114.25) (width 0.25) (layer "F.Cu") (net 2))
   (segment (start 132.6325 114.8525) (end 132.6325 86.36) (width 0.25) (layer "F.Cu") (net 3))
-  (segment (start 134.62 116.84) (end 134.235 117.225) (width 0.25) (layer "F.Cu") (net 3))
   (segment (start 132.6325 86.36) (end 175.26 86.36) (width 0.25) (layer "F.Cu") (net 3))
   (segment (start 134.62 116.84) (end 132.6325 114.8525) (width 0.25) (layer "F.Cu") (net 3))
@@
   (segment (start 92.855 117.765) (end 91.39 116.3) (width 0.25) (layer "F.Cu") (net 4))
   (segment (start 172.72 116.84) (end 136.62 116.84) (width 0.25) (layer "F.Cu") (net 4))
-  (segment (start 91.39 116.775) (end 91.44 116.775) (width 0.25) (layer "F.Cu") (net 4))
-  (segment (start 91.39 116.3) (end 91.39 116.775) (width 0.25) (layer "F.Cu") (net 4))
   (segment (start 175.26 106.68) (end 175.26 116.84) (width 0.25) (layer "F.Cu") (net 5))
 )
